File: projects/module_breakout/module.kicad_pcb (KiCad board)
At the start: 2 copper layers, 25.4 x 52 mm, 6 parts, among them J1 Conn_01x20_Pin, J2 Conn_01x20_Pin, J3 Conn_01x20_Pin, J4 Conn_01x20_Pin

Commit message: RF module test 4
Parts:
- moved J2 7.50 mm to (40.0, 62.0)
Connections:
- J1 pad 11: /A11 -> Net-(J1-Pin_11)
- J1 pad 12: /A12 -> Net-(J1-Pin_12)
- J1 pad 13: /A13 -> Net-(J1-Pin_13)
- J1 pad 14: /A14 -> Net-(J1-Pin_14)
- J1 pad 15: /A15 -> Net-(J1-Pin_15)
- J1 pad 16: /A16 -> Net-(J1-Pin_16)
- J1 pad 17: /A17 -> Net-(J1-Pin_17)
- J1 pad 18: /A18 -> Net-(J1-Pin_18)
- J1 pad 19: /A19 -> Net-(J1-Pin_19)
- J1 pad 20: /A20 -> Net-(J1-Pin_20)
- J2 pad 1: /B1 -> Net-(J2-Pin_1)
- J2 pad 10: /B10 -> Net-(J2-Pin_10)
- J2 pad 2: /B2 -> Net-(J2-Pin_2)
- J2 pad 3: /B3 -> Net-(J2-Pin_3)
- J2 pad 4: /B4 -> Net-(J2-Pin_4)
- J2 pad 5: /B5 -> Net-(J2-Pin_5)
- J2 pad 6: /B6 -> Net-(J2-Pin_6)
- J2 pad 7: /B7 -> Net-(J2-Pin_7)
- J2 pad 8: /B8 -> Net-(J2-Pin_8)
- J2 pad 9: /B9 -> Net-(J2-Pin_9)
- J3 pad 1: Net-(J1-Pin_1) -> Net-(J1-Pin_10)
- J3 pad 10: Net-(J1-Pin_10) -> Net-(J1-Pin_1)
- J3 pad 11: /B1 -> Net-(J2-Pin_10)
- J3 pad 12: /B2 -> Net-(J2-Pin_9)
- J3 pad 13: /B3 -> Net-(J2-Pin_8)
- J3 pad 14: /B4 -> Net-(J2-Pin_7)
- J3 pad 15: /B5 -> Net-(J2-Pin_6)
- J3 pad 16: /B6 -> Net-(J2-Pin_5)
- J3 pad 17: /B7 -> Net-(J2-Pin_4)
- J3 pad 18: /B8 -> Net-(J2-Pin_3)
- J3 pad 19: /B9 -> Net-(J2-Pin_2)
- J3 pad 2: Net-(J1-Pin_2) -> Net-(J1-Pin_9)
- J3 pad 20: /B10 -> Net-(J2-Pin_1)
- J3 pad 3: Net-(J1-Pin_3) -> Net-(J1-Pin_8)
- J3 pad 4: Net-(J1-Pin_4) -> Net-(J1-Pin_7)
- J3 pad 5: Net-(J1-Pin_5) -> Net-(J1-Pin_6)
- J3 pad 6: Net-(J1-Pin_6) -> Net-(J1-Pin_5)
- J3 pad 7: Net-(J1-Pin_7) -> Net-(J1-Pin_4)
- J3 pad 8: Net-(J1-Pin_8) -> Net-(J1-Pin_3)
- J3 pad 9: Net-(J1-Pin_9) -> Net-(J1-Pin_2)
- J4 pad 1: /A11 -> Net-(J1-Pin_20)
- J4 pad 10: /A20 -> Net-(J1-Pin_11)
- J4 pad 11: Net-(J2-Pin_11) -> Net-(J2-Pin_20)
- J4 pad 12: Net-(J2-Pin_12) -> Net-(J2-Pin_19)
- J4 pad 13: Net-(J2-Pin_13) -> Net-(J2-Pin_18)
- J4 pad 14: Net-(J2-Pin_14) -> Net-(J2-Pin_17)
- J4 pad 15: Net-(J2-Pin_15) -> Net-(J2-Pin_16)
- J4 pad 16: Net-(J2-Pin_16) -> Net-(J2-Pin_15)
- J4 pad 17: Net-(J2-Pin_17) -> Net-(J2-Pin_14)
- J4 pad 18: Net-(J2-Pin_18) -> Net-(J2-Pin_13)
- J4 pad 19: Net-(J2-Pin_19) -> Net-(J2-Pin_12)
- J4 pad 2: /A12 -> Net-(J1-Pin_19)
- J4 pad 20: Net-(J2-Pin_20) -> Net-(J2-Pin_11)
- J4 pad 3: /A13 -> Net-(J1-Pin_18)
- J4 pad 4: /A14 -> Net-(J1-Pin_17)
- J4 pad 5: /A15 -> Net-(J1-Pin_16)
- J4 pad 6: /A16 -> Net-(J1-Pin_15)
- J4 pad 7: /A17 -> Net-(J1-Pin_14)
- J4 pad 8: /A18 -> Net-(J1-Pin_13)
- J4 pad 9: /A19 -> Net-(J1-Pin_12)
Routing:
- net /A11: track 41.2 -> 0.00 mm, vias 1 -> 0
- net /B10: track 40.6 -> 0.00 mm, vias 1 -> 0
- net /A12: track 38.1 -> 0.00 mm, vias 1 -> 0
- net /B9: track 37.4 -> 0.00 mm, vias 1 -> 0
- net /A13: track 34.9 -> 0.00 mm, vias 1 -> 0
- net /B8: track 34.2 -> 0.00 mm, vias 1 -> 0
- net /A14: track 31.8 -> 0.00 mm, vias 1 -> 0
- net /B7: track 31.1 -> 0.00 mm, vias 1 -> 0
- net /A15: track 28.6 -> 0.00 mm, vias 1 -> 0
- net /B6: track 27.9 -> 0.00 mm, vias 1 -> 0
- net Net-(J2-Pin_1): track 0.00 -> 26.4 mm
- net /A16: track 26.1 -> 0.00 mm, vias 1 -> 0
- net /B5: track 25.4 -> 0.00 mm, vias 1 -> 0
- net Net-(J2-Pin_2): track 0.00 -> 25.2 mm
- net /A17: track 24.2 -> 0.00 mm, vias 1 -> 0
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Other:
- board text added: "v2"
- board text removed: "v1"
