File: projects/module/module.kicad_pcb (KiCad board)
At the start: 2 copper layers, 70 x 70 mm, 57 parts, among them J1 USB_C, J2 Conn_01x20_Pin, J3 Conn_01x20_Pin, SW1 SW_Push, SW2 SW_Push, U1 RP2040, U2 FLASH, U3 MCP73871, U4 LDK130, U5 ESP32, Y1 12MHz

Commit message: RF module test 9
Parts:
- added R51: 10KΩ, ILO_fp:0402_compact, F.Cu at (68.8, 70.8)
- SW1: value SW_Push -> Button top
- SW2: value SW_Push -> Button side; footprint ILO_fp:Alpsalpine_SKRP_compact -> ILO_fp:Alpsalpine_SKSC
- U4: footprint Package_TO_SOT_SMD:SOT-23-5 -> ILO_fp:SOT-23-5
- moved SW2 27.4 mm to (53.1, 38.5), turned to 180 degrees
- moved SW1 2.55 mm to (52.8, 41.9)
- moved R6 1.91 mm to (50.8, 35.7), turned to 90 degrees
- moved D1 1.56 mm to (51.9, 34.5), turned to -90 degrees
- moved C52 0.75 mm to (68.8, 67.0)
- moved R50 0.75 mm to (68.8, 68.2)
Connections:
- SW2 pad 1: /GP17 -> GND
- SW2 pad 2: GND -> /GP2
- U5 pad 22: unconnected-(U5-IO8-Pad22) -> Net-(U5-IO8/STRAP)
Routing:
- net Net-(U5-IO8/STRAP): track 0.00 -> 15.3 mm, vias 0 -> 2
- net /GP3: track 23.7 -> 21.5 mm
- net /GP17: track 25.5 -> 23.4 mm
- net GND: track 17.9 -> 15.9 mm, vias 27 -> 22
- net /GP25: track 39.1 -> 38.2 mm
- net +3V3: track 94.2 -> 95.1 mm, vias 5 -> 6
- net /GP2: track 19.8 -> 19.0 mm
Other:
- board text added: "ILO RF TEST 9"
- board text removed: "BOOT+"
- board text removed: "ILO RF TEST 8"
