File: projects/module/module.kicad_pcb (KiCad board)
At the start: 2 copper layers, 70 x 70 mm, 58 parts, among them J1 USB_C, J2 Conn_01x20_Pin, J3 Conn_01x20_Pin, SW1 Button top, SW2 Button side, U1 RP2040, U2 FLASH, U3 MCP73871, U4 LDK130, U5 ESP32, Y1 12MHz

Commit message: RF module test 10
Parts:
- added L1: 0.47uH, ILO_fp:0603_compact, F.Cu at (67.5, 44.8)
- C41: value 1uF -> 10uF
- C42: value 1uF -> 22uF
- U4: value LDK130 -> RT6160; footprint ILO_fp:SOT-23-5 -> ILO_fp:WL-CSP-15B-1.4x2.3
- moved C41 3.25 mm to (65.7, 46.4), turned to 90 degrees
- moved C42 3.03 mm to (69.2, 46.4), turned to -90 degrees
- moved REF** 2.10 mm to (64.3, 41.1)
- moved REF** 2.04 mm to (69.1, 43.0)
- moved R34 0.66 mm to (66.1, 42.9), turned to 0 degrees
- moved R33 0.45 mm to (68.8, 42.9), turned to 180 degrees
- moved U4 0.43 mm to (67.5, 46.2), turned to 0 degrees
- moved REF** 0.35 mm to (64.2, 45.2)
- moved REF** 0.11 mm to (62.9, 47.4)
Connections:
- SW2 pad 2: /GP2 -> /RUN
- U3 pad 7: /GP14 -> unconnected-(U3-STAT2-Pad7)
- U3 pad 8: /GP15 -> /GP14
Routing:
- net /RUN: track 11.4 -> 60.8 mm, vias 2 -> 4
- net /GP15: track 25.2 -> 1.61 mm, vias 2 -> 1
- net Net-(L1-Pad2): track 0.00 -> 1.64 mm
- net Net-(L1-Pad1): track 0.00 -> 1.64 mm
- net /GP2: track 19.0 -> 17.4 mm
- net Net-(U3-PROG3): track 4.89 -> 6.26 mm
- net +3V3: track 95.1 -> 93.9 mm
- net VSYS: track 14.1 -> 13.3 mm
- net Net-(U3-THERM): track 3.19 -> 3.84 mm
- net GND: vias 22 -> 23
- removed copper zone on B.Cu, net +3V3
Other:
- board text added: "ILO RF TEST 10"
- board text added: "V-CUT V-CUT V-CUT V-CUT"
- board text removed: "EDGE RAIL V-CUT"
- board text removed: "ILO RF TEST 9"
