File: projects/module/module.kicad_sch (KiCad schematic)
At the start: 55 parts, among them J1 USB_C, J2 Conn_01x20_Pin, J3 Conn_01x20_Pin, SW1 SW_Push, U1 RP2040, U2 FLASH, U3 MCP73871, U4 LDK130, U5 NRF24, Y1 12MHz, Y2 16MHz

Commit message: RF module test 8
Parts:
- removed AE1: Antenna, ILO_fp:Yageo_ANT3216, symbol Device:Antenna
- removed C53: 2.2pF, ILO_fp:0402_compact, symbol Device:C
- removed C54: 4.7pF, ILO_fp:0402_compact, symbol Device:C
- removed C55: 1.5pF, ILO_fp:0402_compact, symbol Device:C
- removed C56: 1pF, ILO_fp:0402_compact, symbol Device:C
- removed C57: 33nF, ILO_fp:0402_compact, symbol Device:C
- removed C58: 1nF, ILO_fp:0402_compact, symbol Device:C
- removed C59: 10nF, ILO_fp:0402_compact, symbol Device:C
- removed L1: 8.2nH, ILO_fp:0402_compact, symbol Device:L
- removed L2: 2.7nH, ILO_fp:0402_compact, symbol Device:L
- removed L3: 3.9nH, ILO_fp:0402_compact, symbol Device:L
- removed R52: 22KΩ, ILO_fp:0402_compact, symbol Device:R
- removed U5: NRF24, ILO_fp:QFN20_internal_routing, symbol ILO_sym:Nordic_nRF24L01
- removed Y2: 16MHz, Crystal:Crystal_SMD_2520-4Pin_2.5x2.0mm, symbol Device:Crystal_GND24
- added C50, C61, C62, C63, C64: 100nF, ILO_fp:0402_compact, symbol Device:C
- added R50: 10KΩ, ILO_fp:0402_compact, symbol Device:R
- added SW2: SW_Push, ILO_fp:Alpsalpine_SKRP_compact, symbol Switch:SW_Push
- added U5: ESP32, ILO_fp:Espressif_ESP32_mini, symbol ILO_sym:Espressif_ESP8684_mini
- C10, C11, C12, C13, C14, C15, C16, C2, C20, C3, C30, C32, C41, C42, C6, C7, C8, C9: Group Capacitor -> C
- C51: value 22pF -> 10uF; Group Capacitor -> C; LCSC C1555 -> C15525
- C52: value 22pF -> 1uF; Group Capacitor -> C; LCSC C1555 -> C52923
- R20, R21, R3, R32, R33, R34, R4, R40, R41, R5, R6: Group Resistor -> R
Connections:
- net +3V3: now also C51.2, C50.2, U5.3 (3V3)
- net ADC0: now also C61.2
- net ADC1: now also C62.2
- net ADC2: now also C63.2
- net ADC3: now also C64.2
- net GND: now also C51.1, C52.1, C50.1, C61.1, C62.1, C63.1, C64.1, SW2.2, U5.0 (GND), U5.1 (GND), U5.11 (GND), U5.14 (GND), U5.2 (GND), U5.36 (GND), U5.37 (GND), U5.38 (GND), U5.39 (GND), U5.40 (GND), U5.41 (GND), U5.42 (GND), U5.43 (GND), U5.44 (GND), U5.45 (GND), U5.46 (GND), U5.47 (GND), U5.48 (GND); no longer C51.2, C52.2, J2.3 (Pin_3), J2.4 (Pin_4), J3.13 (Pin_13), J3.14 (Pin_14), J3.15 (Pin_15), J3.16 (Pin_16)
- net GP17: now also SW2.1, U5.23 (IO9/BOOT)
- net GP25: now also R50.1
- net UART1_RX: now also U5.31 (TXD0)
- net UART1_TX: now also U5.30 (RXD0)
- new net: C52.2, R50.2, U5.8 (EN)
- no-connect marks 5 -> 36
Other:
- note added: "WIRELESS MODULE"
- note removed: "RADIO"
- moved on the sheet: J3

Commit message: RF module test 9
Parts:
- added R51: 10KΩ, ILO_fp:0402_compact, symbol Device:R
- SW1: value SW_Push -> Button top
- SW2: value SW_Push -> Button side; footprint ILO_fp:Alpsalpine_SKRP_compact -> ILO_fp:Alpsalpine_SKSC; LCSC C139797 -> C115362
- U4: footprint Package_TO_SOT_SMD:SOT-23-5 -> ILO_fp:SOT-23-5
- U5: LCSC C3013916 -> C3013915
Connections:
- net +3V3: now also R51.1
- net GND: now also SW2.1; no longer SW2.2
- net GP17: no longer SW2.1
- net GP2: now also SW2.2
- net at U5.22 (IO8/STRAP): now also R51.2
- no-connect marks 36 -> 35
Other:
- moved on the sheet: SW1

Commit message: RF module test 10
Parts:
- removed U4: LDK130, ILO_fp:SOT-23-5, symbol Regulator_Linear:LDK130-33_SOT23_SOT353
- added L1: 0.47uH, ILO_fp:0603_compact, symbol Device:L
- added U4: RT6160, ILO_fp:WL-CSP-15B-1.4x2.3, symbol ILO_sym:Richtek_RT6160
- C41: value 1uF -> 10uF; LCSC C52923 -> C15525
- C42: value 1uF -> 22uF; LCSC C52923 -> C105226
Connections:
- net +3V3: now also U4.E2 (VOUT), U4.E3 (VOUT)
- net GND: now also U4.B1 (VSEL), U4.C1 (AGND), U4.C2 (PGND), U4.C3 (PGND)
- net GP14: now also U3.8 (STAT1); no longer U3.7 (STAT2)
- net GP15: no longer U3.8 (STAT1)
- net GP2: no longer SW2.2
- net RUN: now also SW2.2
- net VSYS: now also U4.A1 (EN), U4.A2 (VIN), U4.A3 (VIN)
- new net: L1.1, U4.B2 (LX1), U4.B3 (LX1)
- new net: L1.2, U4.D2 (LX2), U4.D3 (LX2)
- no-connect marks 35 -> 37
Other:
- moved on the sheet: C30, C32, C41, C42, R32, R33, R34, SW2, U3
